File: cad/LedMatrix.kicad_pcb (KiCad board)
At the start: 2 copper layers, 74 parts, among them J1 Anodes, J2 GNDs

Commit message: initial layout
Parts:
- J1: moved to B.Cu
- moved R8 96.6 mm to (53.3, 85.1)
- moved R7 92.3 mm to (53.3, 77.5)
- moved J1 66.1 mm to (44.5, 50.8), turned to 180 degrees
- moved R6 58.6 mm to (53.3, 69.8)
- moved R5 53.6 mm to (53.3, 62.2)
- moved J2 44.1 mm to (90.2, 21.6), turned to 90 degrees
- moved R4 40.4 mm to (53.3, 54.6)
- moved R3 29.8 mm to (53.3, 47.0)
- moved D21 24.3 mm to (86.4, 62.2)
- moved D29 24.3 mm to (95.2, 62.2)
- moved D37 24.3 mm to (104.1, 62.2)
- moved D45 24.3 mm to (113.0, 62.2)
- moved D53 24.3 mm to (121.9, 62.2)
- moved D61 24.3 mm to (130.8, 62.2)
- moved D13 24.3 mm to (77.5, 62.2)
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
Commit message: compact layout
Parts:
- moved J1 12.7 mm to (57.1, 50.8)
- moved D64 11.4 mm to (120.7, 80.0)
- moved D57 10.9 mm to (120.7, 35.6)
- moved D63 10.9 mm to (120.7, 73.7)
- moved D58 10.5 mm to (120.7, 41.9)
- moved D62 10.5 mm to (120.7, 67.3)
- moved D59 10.2 mm to (120.7, 48.3)
- moved D61 10.2 mm to (120.7, 61.0)
- moved R8 10.2 mm to (62.2, 80.0)
- moved D60 10.2 mm to (120.7, 54.6)
- moved R1 9.67 mm to (62.2, 35.6)
- moved R7 9.67 mm to (62.2, 73.7)
- moved R2 9.25 mm to (62.2, 41.9)
- moved R6 9.25 mm to (62.2, 67.3)
- moved D56 9.16 mm to (114.3, 80.0)
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
Commit message: tracks
Routing:
- net Net-(D57-Pad1): track 0.00 -> 61.6 mm
- net Net-(D1-Pad1): track 0.00 -> 61.0 mm
- net Net-(D1-Pad2): track 0.00 -> 59.1 mm
- net Net-(D16-Pad2): track 0.00 -> 59.1 mm
- net Net-(D15-Pad2): track 0.00 -> 59.0 mm
- net Net-(D10-Pad2): track 0.00 -> 58.9 mm
- net Net-(D13-Pad2): track 0.00 -> 58.9 mm
- net Net-(D12-Pad2): track 0.00 -> 58.9 mm
- net Net-(D11-Pad2): track 0.00 -> 58.9 mm
- net Net-(D14-Pad2): track 0.00 -> 58.9 mm
- net Net-(D49-Pad1): track 0.00 -> 57.8 mm
- net Net-(D10-Pad1): track 0.00 -> 57.5 mm
- net Net-(D41-Pad1): track 0.00 -> 55.4 mm
- net Net-(D17-Pad1): track 0.00 -> 54.2 mm
- net Net-(D33-Pad1): track 0.00 -> 53.8 mm
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
Commit message: board outline
Parts:
- added REF**: MountingHole_2.5mm, MountingHole:MountingHole_2.5mm, F.Cu at (58.4, 85.1)
- added REF**: MountingHole_2.5mm, MountingHole:MountingHole_2.5mm, F.Cu at (127.0, 85.1)
- added REF**: MountingHole_2.5mm, MountingHole:MountingHole_2.5mm, F.Cu at (127.0, 29.2)
- added REF**: MountingHole_2.5mm, MountingHole:MountingHole_2.5mm, F.Cu at (58.4, 29.2)
- J1, J2: footprint Connector_PinHeader_2.54mm:PinHeader_1x08_P2.54mm_Horizontal -> Connector_PinHeader_2.54mm:PinHeader_1x08_P2.54mm_Vertical
Other:
- board outline added: 76.2 x 63.5 mm
- board text added: "LED Matrix v1.0 (c) 2019 Steve"

Commit message: gerbers
Parts:
- removed REF** (x4): MountingHole_2.5mm, MountingHole:MountingHole_2.5mm
Changed lines of the file:
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@@
     (tracks 320)
     (zones 0)
-    (modules 78)
+    (modules 74)
     (nets 25)
   )
@@
     (add_net "Net-(J1-Pad8)")
   )
-  (module MountingHole:MountingHole_2.5mm (layer F.Cu)
-    (at 58.42 85.09)
-    (descr "Mounting Hole 2.5mm, no annular")
-    (tags "mounting hole 2.5mm no annular")
-    (attr virtual)
-    (fp_text reference REF** (at 0 -3.5) (layer F.SilkS) hide
-      (effects (font (size 1 1) (thickness 0.15)))
-    )
-    (fp_text value MountingHole_2.5mm (at 0 3.5) (layer F.Fab) hide
-      (effects (font (size 1 1) (thickness 0.15)))
-    )
-    (fp_text user %R (at 0.3 0) (layer F.Fab)
-      (effects (font (size 1 1) (thickness 0.15)))
-    )
-    (fp_circle (center 0 0) (end 2.5 0) (layer Cmts.User) (width 0.15))
-    (fp_circle (center 0 0) (end 2.75 0) (layer F.CrtYd) (width 0.05))
-    (pad "" np_thru_hole circle (at 0 0) (size 2.5 2.5) (drill 2.5) (layers *.Cu *.Mask))
-  )
-  (module MountingHole:MountingHole_2.5mm (layer F.Cu)
-    (at 127 85.09)
-    (descr "Mounting Hole 2.5mm, no annular")
-    (tags "mounting hole 2.5mm no annular")
-    (attr virtual)
-    (fp_text reference REF** (at 0 -3.5) (layer F.SilkS) hide
-      (effects (font (size 1 1) (thickness 0.15)))
-    )
-    (fp_text value MountingHole_2.5mm (at 0 3.5) (layer F.Fab) hide
-      (effects (font (size 1 1) (thickness 0.15)))
-    )
-    (fp_circle (center 0 0) (end 2.75 0) (layer F.CrtYd) (width 0.05))
-    (fp_circle (center 0 0) (end 2.5 0) (layer Cmts.User) (width 0.15))
-    (fp_text user %R (at 0.3 0) (layer F.Fab)
-      (effects (font (size 1 1) (thickness 0.15)))
-    )
-    (pad "" np_thru_hole circle (at 0 0) (size 2.5 2.5) (drill 2.5) (layers *.Cu *.Mask))
-  )
-  (module MountingHole:MountingHole_2.5mm (layer F.Cu)
-    (at 127 29.21)
-    (descr "Mounting Hole 2.5mm, no annular")
-    (tags "mounting hole 2.5mm no annular")
-    (attr virtual)
-    (fp_text reference REF** (at 0 -3.5) (layer F.SilkS) hide
-      (effects (font (size 1 1) (thickness 0.15)))
-    )
-    (fp_text value MountingHole_2.5mm (at 0 3.5) (layer F.Fab) hide
-      (effects (font (size 1 1) (thickness 0.15)))
-    )
-    (fp_text user %R (at 0.3 0) (layer F.Fab)
-      (effects (font (size 1 1) (thickness 0.15)))
-    )
-    (fp_circle (center 0 0) (end 2.5 0) (layer Cmts.User) (width 0.15))
-    (fp_circle (center 0 0) (end 2.75 0) (layer F.CrtYd) (width 0.05))
-    (pad "" np_thru_hole circle (at 0 0) (size 2.5 2.5) (drill 2.5) (layers *.Cu *.Mask))
-  )
   (module Connector_PinHeader_2.54mm:PinHeader_1x08_P2.54mm_Vertical (layer F.Cu)
     (at 88.9 27.94 90)
@@
     )
   )
-  (module MountingHole:MountingHole_2.5mm (layer F.Cu)
-    (at 58.42 29.21)
-    (descr "Mounting Hole 2.5mm, no annular")
-    (tags "mounting hole 2.5mm no annular")
-    (attr virtual)
-    (fp_text reference REF** (at 0 -3.5) (layer F.SilkS) hide
-      (effects (font (size 1 1) (thickness 0.15)))
-    )
-    (fp_text value MountingHole_2.5mm (at 0 3.5) (layer F.Fab) hide
-      (effects (font (size 1 1) (thickness 0.15)))
-    )
-    (fp_circle (center 0 0) (end 2.75 0) (layer F.CrtYd) (width 0.05))
-    (fp_circle (center 0 0) (end 2.5 0) (layer Cmts.User) (width 0.15))
-    (fp_text user %R (at 0.3 0) (layer F.Fab)
-      (effects (font (size 1 1) (thickness 0.15)))
-    )
-    (pad "" np_thru_hole circle (at 0 0) (size 2.5 2.5) (drill 2.5) (layers *.Cu *.Mask))
-  )
   (dimension 63.5 (width 0.3) (layer F.Fab)
