File: cad/LedMatrix.sch (KiCad schematic (older format))
At the start: 74 parts, among them J1 Rows, J2 Columns

Commit message: add netlist
Parts:
- D1, D10, D11, D12, D13, D14, D15, D16, D17, D18, D19, D2, D20, D21, D22, D23, D24, D25, D26, D27, D28, D29, D3, D30, D31, D32, D33, D34, D35, D36, D37, D38, D39, D4, D40, D41, D42, D43, D44, D45, D46, D47, D48, D49, D5, D50, D51, D52, D53, D54, D55, D56, D57, D58, D59, D6, D60, D61, D62, D63, D64, D7, D8, D9: footprint (none) -> LED_THT:LED_D3.0mm
- J1: value Rows -> Anodes; footprint (none) -> Connector_PinHeader_2.54mm:PinHeader_1x08_P2.54mm_Horizontal
- J2: value Columns -> GNDs; footprint (none) -> Connector_PinHeader_2.54mm:PinHeader_1x08_P2.54mm_Horizontal
- R1, R2, R3, R4, R5, R6, R7, R8: footprint (none) -> Resistor_THT:R_Axial_DIN0207_L6.3mm_D2.5mm_P10.16mm_Horizontal

Commit message: ...
Other:
- note added: "1.0"
- note added: "Simple 8x8 LED Matrix"
Changed lines of the file:
@@
 Wire Wire Line
 	5050 6300 5050 6650
+Text Notes 7550 7500 0    50   ~ 10
+Simple 8x8 LED Matrix
+Text Notes 10650 7650 0    50   ~ 10
+1.0
 $EndSCHEMATC

Commit message: board outline
Parts:
- J1, J2: footprint Connector_PinHeader_2.54mm:PinHeader_1x08_P2.54mm_Horizontal -> Connector_PinHeader_2.54mm:PinHeader_1x08_P2.54mm_Vertical
Changed lines of the file:
@@
 F 0 "J1" H 1744 4335 50  0000 C CNN
 F 1 "Anodes" H 1744 4244 50  0000 C CNN
-F 2 "Connector_PinHeader_2.54mm:PinHeader_1x08_P2.54mm_Horizontal" H 1850 3850 50  0001 C CNN
+F 2 "Connector_PinHeader_2.54mm:PinHeader_1x08_P2.54mm_Vertical" H 1850 3850 50  0001 C CNN
 F 3 "~" H 1850 3850 50  0001 C CNN
 	1    1850 3850
@@
 F 0 "J2" V 5272 7280 50  0000 C CNN
 F 1 "GNDs" V 5363 7280 50  0000 C CNN
-F 2 "Connector_PinHeader_2.54mm:PinHeader_1x08_P2.54mm_Horizontal" H 5200 7350 50  0001 C CNN
+F 2 "Connector_PinHeader_2.54mm:PinHeader_1x08_P2.54mm_Vertical" H 5200 7350 50  0001 C CNN
 F 3 "~" H 5200 7350 50  0001 C CNN
 	1    5200 7350

Commit message: gerbers
Other:
- note removed: "1.0"
- note removed: "Simple 8x8 LED Matrix"
Changed lines of the file:
@@
 encoding utf-8
 Sheet 1 1
-Title ""
-Date ""
-Rev ""
-Comp ""
+Title "8x8 LED Matrix"
+Date "2019-05-25"
+Rev "1.0"
+Comp "Stephen Crane"
 Comment1 ""
 Comment2 ""
@@
 Wire Wire Line
 	5050 6300 5050 6650
-Text Notes 7550 7500 0    50   ~ 10
-Simple 8x8 LED Matrix
-Text Notes 10650 7650 0    50   ~ 10
-1.0
 $EndSCHEMATC
